File: pcb/pcb.sch (KiCad schematic (older format))
At the start: 9 parts

Commit message: Completed schematics
Parts:
- BZ1: renamed from BZ?; footprint (none) -> Buzzer_Beeper:Buzzer_TDK_PS1240P02BT_D12.2mm_H6.5mm
- R1, R2, R3, R4, R5: renamed from R?; footprint (none) -> Resistor_THT:R_Axial_DIN0207_L6.3mm_D2.5mm_P15.24mm_Horizontal
- SW1: renamed from SW?; footprint (none) -> Button_Switch_THT:SW_PUSH_6mm_H4.3mm
- gave numbers to parts that had none: 2
Connections:
- net +5V: now also R2.2; no longer R2.1
- net GND: now also U1.16 (K)
- net KEY_POS: no longer A1.6 (D3), R5.2, SW1.2
- net at A1.10 (D7): now also U1.11 (DB4)
- net at A1.11 (D8): now also U1.12 (DB5)
- net at A1.12 (D9): now also U1.13 (DB6)
- net at A1.13 (D10): now also U1.14 (DB7)
- net at A1.9 (D6): now also U1.6 (E)
- net at U1.15 (A/VEE): now also R2.1
- new net: A1.6 (D3), R5.2, SW1.2
Other:
- moved on the sheet: R2
Changed lines of the file:
@@
 	6750 4050 6750 4100
 $Comp
-L power:GND #PWR?
+L power:GND #PWR013
 U 1 1 5EE31265
 P 6950 4150
-F 0 "#PWR?" H 6950 3900 50  0001 C CNN
+F 0 "#PWR013" H 6950 3900 50  0001 C CNN
 F 1 "GND" H 6955 3977 50  0000 C CNN
 F 2 "" H 6950 4150 50  0001 C CNN
@@
 $EndComp
 $Comp
-L MCU_Module:Arduino_Nano_v3.x A?
+L MCU_Module:Arduino_Nano_v3.x A1
 U 1 1 5ED974A3
 P 6650 3050
-F 0 "A?" H 6650 1961 50  0000 C CNN
+F 0 "A1" H 6650 1961 50  0000 C CNN
 F 1 "Arduino_Nano_v3.x" H 6450 1900 50  0000 C CNN
 F 2 "Module:Arduino_Nano" H 6650 3050 50  0001 C CIN
@@
 	6850 2050 6850 1850
 $Comp
-L power:+5V #PWR?
+L power:+5V #PWR012
 U 1 1 5EE2FDF2
 P 6850 1850
-F 0 "#PWR?" H 6850 1700 50  0001 C CNN
+F 0 "#PWR012" H 6850 1700 50  0001 C CNN
 F 1 "+5V" H 6865 2023 50  0000 C CNN
 F 2 "" H 6850 1850 50  0001 C CNN
@@
 	5800 2200 5800 2100
 $Comp
-L power:+5V #PWR?
+L power:+5V #PWR09
 U 1 1 5EE2C21F
 P 5800 2100
-F 0 "#PWR?" H 5800 1950 50  0001 C CNN
+F 0 "#PWR09" H 5800 1950 50  0001 C CNN
 F 1 "+5V" H 5815 2273 50  0000 C CNN
 F 2 "" H 5800 2100 50  0001 C CNN
@@
 $EndComp
 Wire Wire Line
-	5800 2500 5800 2750
-Connection ~ 5800 2850
-Wire Wire Line
 	5950 2750 6150 2750
-Connection ~ 5950 2750
 Wire Wire Line
 	5950 2500 5950 2750
 Wire Wire Line
-	5800 2750 5950 2750
-Wire Wire Line
 	5800 2850 6150 2850
 Wire Wire Line
@@
 	5750 3100 5800 3100
 $Comp
-L Device:R R?
+L Device:R R4
 U 1 1 5EDA79C7
 P 5800 2350
-F 0 "R?" H 5731 2304 50  0000 R CNN
+F 0 "R4" H 5731 2304 50  0000 R CNN
 F 1 "470" H 5731 2395 50  0000 R CNN
-F 2 "" V 5730 2350 50  0001 C CNN
+F 2 "Resistor_THT:R_Axial_DIN0207_L6.3mm_D2.5mm_P15.24mm_Horizontal" V 5730 2350 50  0001 C CNN
 F 3 "~" H 5800 2350 50  0001 C CNN
 	1    5800 2350
@@
 	5950 2200 5950 2100
 $Comp
-L Device:R R?
+L Device:R R5
 U 1 1 5EE023BD
 P 5950 2350
-F 0 "R?" H 6020 2396 50  0000 L CNN
+F 0 "R5" H 6020 2396 50  0000 L CNN
 F 1 "470" H 6020 2305 50  0000 L CNN
-F 2 "" V 5880 2350 50  0001 C CNN
+F 2 "Resistor_THT:R_Axial_DIN0207_L6.3mm_D2.5mm_P15.24mm_Horizontal" V 5880 2350 50  0001 C CNN
 F 3 "~" H 5950 2350 50  0001 C CNN
 	1    5950 2350
@@
 	5350 2800 5350 2750
 $Comp
-L power:GND #PWR?
+L power:GND #PWR07
 U 1 1 5EDE763B
 P 5350 2800
-F 0 "#PWR?" H 5350 2550 50  0001 C CNN
+F 0 "#PWR07" H 5350 2550 50  0001 C CNN
 F 1 "GND" H 5355 2627 50  0000 C CNN
 F 2 "" H 5350 2800 50  0001 C CNN
@@
 $EndComp
 $Comp
-L power:+5V #PWR?
+L power:+5V #PWR010
 U 1 1 5EDE60D0
 P 5950 2100
-F 0 "#PWR?" H 5950 1950 50  0001 C CNN
+F 0 "#PWR010" H 5950 1950 50  0001 C CNN
 F 1 "+5V" H 5965 2273 50  0000 C CNN
 F 2 "" H 5950 2100 50  0001 C CNN
@@
 $EndComp
 $Comp
-L Switch:SW_Push SW?
+L Switch:SW_Push SW1
 U 1 1 5EDDEC17
 P 5600 2750
-F 0 "SW?" H 5600 2700 50  0000 C CNN
+F 0 "SW1" H 5600 2700 50  0000 C CNN
 F 1 "SW_Push" H 5600 2600 50  0000 C CNN
-F 2 "" H 5600 2950 50  0001 C CNN
+F 2 "Button_Switch_THT:SW_PUSH_6mm_H4.3mm" H 5600 2950 50  0001 C CNN
 F 3 "~" H 5600 2950 50  0001 C CNN
 	1    5600 2750
@@
 	4850 2850 4950 2850
 $Comp
-L power:GND #PWR?
+L power:GND #PWR06
 U 1 1 5EDB1E9C
 P 4950 3300
-F 0 "#PWR?" H 4950 3050 50  0001 C CNN
+F 0 "#PWR06" H 4950 3050 50  0001 C CNN
 F 1 "GND" H 4955 3127 50  0000 C CNN
 F 2 "" H 4950 3300 50  0001 C CNN
@@
 $EndComp
 $Comp
-L Device:R R?
+L Device:R R3
 U 1 1 5EDA738A
 P 4950 3050
-F 0 "R?" H 5020 3096 50  0000 L CNN
+F 0 "R3" H 5020 3096 50  0000 L CNN
 F 1 "470" H 5020 3005 50  0000 L CNN
-F 2 "" V 4880 3050 50  0001 C CNN
+F 2 "Resistor_THT:R_Axial_DIN0207_L6.3mm_D2.5mm_P15.24mm_Horizontal" V 4880 3050 50  0001 C CNN
 F 3 "~" H 4950 3050 50  0001 C CNN
 	1    4950 3050
@@
 $EndComp
 $Comp
-L Device:Buzzer BZ?
+L Device:Buzzer BZ1
 U 1 1 5ED9989F
 P 4750 2750
-F 0 "BZ?" H 4902 2779 50  0000 L CNN
+F 0 "BZ1" H 4902 2779 50  0000 L CNN
 F 1 "Buzzer" H 4902 2688 50  0000 L CNN
-F 2 "" V 4725 2850 50  0001 C CNN
+F 2 "Buzzer_Beeper:Buzzer_TDK_PS1240P02BT_D12.2mm_H6.5mm" V 4725 2850 50  0001 C CNN
 F 3 "~" V 4725 2850 50  0001 C CNN
 	1    4750 2750
 	-1   0    0    -1
 $EndComp
-Text GLabel 3800 5500 0    50   Input ~ 0
+Text GLabel 6650 4700 0    50   Input ~ 0
 KEY_NEG
 $Comp
-L power:GND #PWR?
+L power:GND #PWR011
 U 1 1 5EE65809
-P 3950 5550
-F 0 "#PWR?" H 3950 5300 50  0001 C CNN
-F 1 "GND" H 3955 5377 50  0000 C CNN
-F 2 "" H 3950 5550 50  0001 C CNN
-F 3 "" H 3950 5550 50  0001 C CNN
-	1    3950 5550
-	1    0    0    -1
-$EndComp
-Wire Wire Line
-	3800 5500 3950 5500
-Wire Wire Line
-	3950 5500 3950 5550
-Connection ~ 5800 2750
-Wire Wire Line
-	5800 2750 5800 2850
-$Comp
-L Device:R R?
+P 6800 4750
+F 0 "#PWR011" H 6800 4500 50  0001 C CNN
+F 1 "GND" H 6805 4577 50  0000 C CNN
+F 2 "" H 6800 4750 50  0001 C CNN
+F 3 "" H 6800 4750 50  0001 C CNN
+	1    6800 4750
+	1    0    0    -1
+$EndComp
+Wire Wire Line
+	6650 4700 6800 4700
+Wire Wire Line
+	6800 4700 6800 4750
+$Comp
+L Device:R R1
 U 1 1 5EDA6D10
 P 3650 3950
-F 0 "R?" V 3443 3950 50  0000 C CNN
+F 0 "R1" V 3443 3950 50  0000 C CNN
 F 1 "3.3K" V 3534 3950 50  0000 C CNN
-F 2 "" V 3580 3950 50  0001 C CNN
+F 2 "Resistor_THT:R_Axial_DIN0207_L6.3mm_D2.5mm_P15.24mm_Horizontal" V 3580 3950 50  0001 C CNN
 F 3 "~" H 3650 3950 50  0001 C CNN
 	1    3650 3950
@@
 $EndComp
 $Comp
-L Device:R R?
+L Device:R R2
 U 1 1 5EDA7700
-P 5350 5100
-F 0 "R?" V 5150 5100 50  0000 C CNN
-F 1 "470" V 5250 5100 50  0000 C CNN
-F 2 "" V 5280 5100 50  0001 C CNN
-F 3 "~" H 5350 5100 50  0001 C CNN
-	1    5350 5100
-	0    1    1    0
-$EndComp
-$Comp
-L power:GND #PWR?
+P 4500 4050
+F 0 "R2" V 4300 4050 50  0000 C CNN
+F 1 "470" V 4400 4050 50  0000 C CNN
+F 2 "Resistor_THT:R_Axial_DIN0207_L6.3mm_D2.5mm_P15.24mm_Horizontal" V 4430 4050 50  0001 C CNN
+F 3 "~" H 4500 4050 50  0001 C CNN
+	1    4500 4050
+	0    -1   1    0
+$EndComp
+$Comp
+L power:GND #PWR08
 U 1 1 5EDB1113
 P 5400 4600
-F 0 "#PWR?" H 5400 4350 50  0001 C CNN
+F 0 "#PWR08" H 5400 4350 50  0001 C CNN
 F 1 "GND" H 5405 4427 50  0000 C CNN
 F 2 "" H 5400 4600 50  0001 C CNN
@@
 $EndComp
 $Comp
-L Display_Character:LCD-016N002L U?
+L Display_Character:LCD-016N002L U1
 U 1 1 5ED98DC7
 P 4500 4550
-F 0 "U?" V 4850 5350 50  0000 R CNN
+F 0 "U1" V 4850 5350 50  0000 R CNN
 F 1 "LCD-016N002L" V 4850 4100 50  0000 R CNN
 F 2 "Display:LCD-016N002L" H 4520 3630 50  0001 C CNN
@@
 	5400 4550 5400 4600
 $Comp
-L power:+5V #PWR?
+L power:+5V #PWR02
 U 1 1 5EE6A5F3
 P 3600 4450
-F 0 "#PWR?" H 3600 4300 50  0001 C CNN
+F 0 "#PWR02" H 3600 4300 50  0001 C CNN
 F 1 "+5V" H 3615 4623 50  0000 C CNN
 F 2 "" H 3600 4450 50  0001 C CNN
@@
 	3600 4550 3600 4450
 $Comp
-L power:GND #PWR?
+L power:GND #PWR01
 U 1 1 5EE7CD7F
 P 3450 4050
-F 0 "#PWR?" H 3450 3800 50  0001 C CNN
+F 0 "#PWR01" H 3450 3800 50  0001 C CNN
 F 1 "GND" H 3455 3877 50  0000 C CNN
 F 2 "" H 3450 4050 50  0001 C CNN
@@
 Wire Wire Line
 	3450 3950 3500 3950
-Wire Wire Line
-	5100 4950 5100 5100
-Wire Wire Line
-	5100 5100 5200 5100
-$Comp
-L power:+5V #PWR?
+$Comp
+L power:+5V #PWR05
 U 1 1 5EE91567
-P 5550 5000
-F 0 "#PWR?" H 5550 4850 50  0001 C CNN
-F 1 "+5V" H 5565 5173 50  0000 C CNN
-F 2 "" H 5550 5000 50  0001 C CNN
-F 3 "" H 5550 5000 50  0001 C CNN
-	1    5550 5000
-	1    0    0    -1
-$EndComp
-Wire Wire Line
-	5500 5100 5550 5100
-Wire Wire Line
-	5550 5100 5550 5000
-$Comp
-L power:GND #PWR?
+P 4700 4000
+F 0 "#PWR05" H 4700 3850 50  0001 C CNN
+F 1 "+5V" H 4715 4173 50  0000 C CNN
+F 2 "" H 4700 4000 50  0001 C CNN
+F 3 "" H 4700 4000 50  0001 C CNN
+	1    4700 4000
+	1    0    0    -1
+$EndComp
+$Comp
+L power:GND #PWR03
 U 1 1 5EE976E1
 P 4000 5050
-F 0 "#PWR?" H 4000 4800 50  0001 C CNN
+F 0 "#PWR03" H 4000 4800 50  0001 C CNN
 F 1 "GND" H 4005 4877 50  0000 C CNN
 F 2 "" H 4000 5050 50  0001 C CNN
@@
 Wire Wire Line
 	5900 2950 6150 2950
+Connection ~ 5800 2850
+Connection ~ 5950 2750
+Wire Wire Line
+	5800 2750 5950 2750
+Wire Wire Line
+	5800 2500 5800 2850
+Wire Wire Line
+	3900 4950 3900 5200
+Wire Wire Line
+	3900 5200 3350 5200
+Wire Wire Line
+	3350 5200 3350 3550
+Wire Wire Line
+	3350 3550 6000 3550
+Wire Wire Line
+	6000 3550 6000 3050
+Wire Wire Line
+	6000 3050 6150 3050
+Wire Wire Line
+	4800 4950 4800 5300
+Wire Wire Line
+	4800 5300 5800 5300
+Wire Wire Line
+	5800 5300 5800 3150
+Wire Wire Line
+	5800 3150 6150 3150
+Wire Wire Line
+	4900 4950 4900 5400
+Wire Wire Line
+	4900 5400 5700 5400
+Wire Wire Line
+	5700 5400 5700 3250
+Wire Wire Line
+	5700 3250 6150 3250
+Wire Wire Line
+	5000 4950 5000 5500
+Wire Wire Line
+	5000 5500 5600 5500
+Wire Wire Line
+	5600 5500 5600 3350
+Wire Wire Line
+	5600 3350 6150 3350
+Wire Wire Line
+	4200 4150 4200 4050
+Wire Wire Line
+	4650 4050 4700 4050
+Wire Wire Line
+	4700 4050 4700 4000
+Wire Wire Line
+	5100 4950 5100 5200
+Wire Wire Line
+	5100 5200 5500 5200
+Wire Wire Line
+	5500 5200 5500 3450
+Wire Wire Line
+	5500 3450 6150 3450
+Wire Wire Line
+	4200 4050 4350 4050
+$Comp
+L power:GND #PWR04
+U 1 1 5EDD6538
+P 4050 3950
+F 0 "#PWR04" H 4050 3700 50  0001 C CNN
+F 1 "GND" H 4055 3777 50  0000 C CNN
+F 2 "" H 4050 3950 50  0001 C CNN
+F 3 "" H 4050 3950 50  0001 C CNN
+	1    4050 3950
+	1    0    0    -1
+$EndComp
+Wire Wire Line
+	4050 3950 4050 3900
+Wire Wire Line
+	4050 3900 4300 3900
+Wire Wire Line
+	4300 3900 4300 4150
 $EndSCHEMATC

Commit message: Finished schematics and added pcb layout
Parts:
- added J1: Audio Jack, Connector_Audio:Jack_3.5mm_Ledino_KB3SPRS_Horizontal, symbol AudioJackCustom:AudioJack2_Dual_Ground_Switch
Connections:
- net GND: now also J1.S
- net KEY_POS: now also J1.T
Changed lines of the file:
@@
 	-1   0    0    -1
 $EndComp
-Text GLabel 6650 4700 0    50   Input ~ 0
+Text GLabel 6700 5300 0    50   Input ~ 0
 KEY_NEG
 $Comp
 L power:GND #PWR011
 U 1 1 5EE65809
-P 6800 4750
-F 0 "#PWR011" H 6800 4500 50  0001 C CNN
-F 1 "GND" H 6805 4577 50  0000 C CNN
-F 2 "" H 6800 4750 50  0001 C CNN
-F 3 "" H 6800 4750 50  0001 C CNN
-	1    6800 4750
-	1    0    0    -1
-$EndComp
-Wire Wire Line
-	6650 4700 6800 4700
-Wire Wire Line
-	6800 4700 6800 4750
+P 6850 5350
+F 0 "#PWR011" H 6850 5100 50  0001 C CNN
+F 1 "GND" H 6855 5177 50  0000 C CNN
+F 2 "" H 6850 5350 50  0001 C CNN
+F 3 "" H 6850 5350 50  0001 C CNN
+	1    6850 5350
+	1    0    0    -1
+$EndComp
+Wire Wire Line
+	6700 5300 6850 5300
+Wire Wire Line
+	6850 5300 6850 5350
 $Comp
 L Device:R R1
@@
 Wire Wire Line
 	4300 3900 4300 4150
+$Comp
+L AudioJackCustom:AudioJack2_Dual_Ground_Switch J1
+U 1 1 5EDF1D17
+P 6400 4750
+F 0 "J1" H 6350 5200 50  0000 C CNN
+F 1 "Audio Jack" H 6400 5100 50  0000 C CNN
+F 2 "Connector_Audio:Jack_3.5mm_Ledino_KB3SPRS_Horizontal" H 6350 4950 50  0001 C CNN
+F 3 "~" H 6350 4950 50  0001 C CNN
+	1    6400 4750
+	1    0    0    -1
+$EndComp
+Text GLabel 6500 5100 2    50   Input ~ 0
+KEY_NEG
+Wire Wire Line
+	6400 5050 6400 5100
+Wire Wire Line
+	6400 5100 6500 5100
+Text GLabel 6700 4750 2    50   Input ~ 0
+KEY_POS
+Wire Wire Line
+	6600 4750 6700 4750
 $EndSCHEMATC

Commit message: Finished pcb wiring
Changed lines of the file:
@@
 	-1   0    0    -1
 $EndComp
-Text GLabel 6700 5300 0    50   Input ~ 0
-KEY_NEG
 $Comp
 L power:GND #PWR011
 U 1 1 5EE65809
-P 6850 5350
-F 0 "#PWR011" H 6850 5100 50  0001 C CNN
-F 1 "GND" H 6855 5177 50  0000 C CNN
-F 2 "" H 6850 5350 50  0001 C CNN
-F 3 "" H 6850 5350 50  0001 C CNN
-	1    6850 5350
-	1    0    0    -1
-$EndComp
-Wire Wire Line
-	6700 5300 6850 5300
-Wire Wire Line
-	6850 5300 6850 5350
+P 6550 5150
+F 0 "#PWR011" H 6550 4900 50  0001 C CNN
+F 1 "GND" H 6555 4977 50  0000 C CNN
+F 2 "" H 6550 5150 50  0001 C CNN
+F 3 "" H 6550 5150 50  0001 C CNN
+	1    6550 5150
+	1    0    0    -1
+$EndComp
 $Comp
 L Device:R R1
@@
 	1    0    0    -1
 $EndComp
-Text GLabel 6500 5100 2    50   Input ~ 0
-KEY_NEG
-Wire Wire Line
-	6400 5050 6400 5100
-Wire Wire Line
-	6400 5100 6500 5100
 Text GLabel 6700 4750 2    50   Input ~ 0
 KEY_POS
 Wire Wire Line
 	6600 4750 6700 4750
+Wire Wire Line
+	6400 5050 6400 5100
+Wire Wire Line
+	6400 5100 6550 5100
+Wire Wire Line
+	6550 5100 6550 5150
 $EndSCHEMATC

Commit message: Redesigned pcb due to a bug
Parts:
- U1: footprint Display:LCD-016N002L -> Display:WC1602A
Changed lines of the file:
@@
 F 0 "U1" V 4850 5350 50  0000 R CNN
 F 1 "LCD-016N002L" V 4850 4100 50  0000 R CNN
-F 2 "Display:LCD-016N002L" H 4520 3630 50  0001 C CNN
+F 2 "Display:WC1602A" H 4520 3630 50  0001 C CNN
 F 3 "http://www.vishay.com/docs/37299/37299.pdf" H 5000 4250 50  0001 C CNN
 	1    4500 4550

Commit message: Update pin numbers
Parts:
- BZ1: footprint Buzzer_Beeper:Buzzer_TDK_PS1240P02BT_D12.2mm_H6.5mm -> Buzzer_Beeper:MagneticBuzzer_Kingstate_KCG0601
Changed lines of the file:
@@
 F 0 "BZ1" H 4902 2779 50  0000 L CNN
 F 1 "Buzzer" H 4902 2688 50  0000 L CNN
-F 2 "Buzzer_Beeper:Buzzer_TDK_PS1240P02BT_D12.2mm_H6.5mm" V 4725 2850 50  0001 C CNN
+F 2 "Buzzer_Beeper:MagneticBuzzer_Kingstate_KCG0601" V 4725 2850 50  0001 C CNN
 F 3 "~" V 4725 2850 50  0001 C CNN
 	1    4750 2750

Commit message: Updated a footprint
Parts:
- BZ1: footprint Buzzer_Beeper:MagneticBuzzer_Kingstate_KCG0601 -> Buzzer_Beeper:Buzzer_TDK_PS1240P02BT_D12.2mm_H6.5mm
Changed lines of the file:
@@
 F 0 "BZ1" H 4902 2779 50  0000 L CNN
 F 1 "Buzzer" H 4902 2688 50  0000 L CNN
-F 2 "Buzzer_Beeper:MagneticBuzzer_Kingstate_KCG0601" V 4725 2850 50  0001 C CNN
+F 2 "Buzzer_Beeper:Buzzer_TDK_PS1240P02BT_D12.2mm_H6.5mm" V 4725 2850 50  0001 C CNN
 F 3 "~" V 4725 2850 50  0001 C CNN
 	1    4750 2750
